Commit message: modified

File: urdf/base/base_mp500.urdf.xacro (robot description, xacro)
@@ -29,14 +29,15 @@
 			<geometry>
 				<mesh filename="package://mp500lwa4d_description/meshes/mp500/MP500-BODY.STL" scale="0.01 0.01 0.01"/>
-			<!--cylinder length="0.381" radius="0.2545"/-->
-			<!--box size="0.445 0.277 0.17"/-->
+				<!--cylinder length="0.381" radius="0.2545"/-->
+				<!--box size="0.445 0.277 0.17"/-->
 			</geometry>
 			<material name="Grey" />
 		</visual>
 		<collision name='body_collision'>
-			<origin xyz="0 0 0.216" rpy="0 0 -1.57" />
+			<origin xyz="-0.160 0.0 0.09" rpy="0 0 -1.57" />
 			<geometry>
-				<box size="0.400 0.676 0.300"/>
-				<!--cylinder length="0.381" radius="0.2545"/-->
+				<mesh filename="package://mp500lwa4d_description/meshes/mp500/MP500-BODY.STL" scale="0.01 0.01 0.01"/>
+				<!--box size="0.400 0.676 0.300"/>
+				<cylinder length="0.381" radius="0.2545"/-->
 			</geometry>
 		</collision>
@@ -57,8 +58,9 @@
 		</visual>
 		<collision>
-			<origin xyz="0 0 0" rpy="0 1.57 -1.57" />
+			<origin xyz="0 0 0" rpy="0 0 -1.57" />
 			<geometry>
-				<cylinder radius="0.125" length="0.085"/>
-		</geometry>
+				<mesh filename="package://mp500lwa4d_description/meshes/mp500/MP500-WHEEL.STL" scale="0.01 0.01 0.01" />
+				<!--cylinder radius="0.125" length="0.085"/-->
+			</geometry>
 		</collision>
 	</link>
@@ -116,7 +118,8 @@
 		</visual>
 		<collision>
-			<origin xyz="0 0 0" rpy="0 1.57 -1.57" />
+			<origin xyz="0 0 0" rpy="0 0 -1.57" />
 			<geometry>
-				<cylinder radius="0.125" length="0.085"/>
+				<mesh filename="package://mp500lwa4d_description/meshes/mp500/MP500-WHEEL.STL" scale="0.01 0.01 0.01" />
+				<!--cylinder radius="0.125" length="0.085"/-->
 			</geometry>
 		</collision>
@@ -148,5 +151,6 @@
 			<origin xyz="0 0 0" rpy="0 0 -1.57" />
 			<geometry>
-				<sphere radius="0.00115"/>
+				<mesh filename="package://mp500lwa4d_description/meshes/mp500/HANGER-WHEEL.STL" scale="0.01 0.01 0.01" />
+				<!--sphere radius="0.00115"/-->
 			</geometry>
 		</collision>

File: urdf/robot.gazebo.xacro (robot description, xacro)
@@ -3,5 +3,5 @@
     <gazebo>
         <plugin name="differential_drive_controller" filename="libgazebo_ros_diff_drive.so">
-        <robotNamespace>/mp500lwa4d</robotNamespace>
+        <robotNamespace>/</robotNamespace>
         <alwaysOn>true</alwaysOn>
         <updateRate>50</updateRate>

File: urdf/sensor/rplidar.urdf.xacro (robot description, xacro)
@@ -18,13 +18,14 @@
 				<origin xyz="0 0 -0.04" rpy="3.14 0 -1.57" />
 				<geometry>
-                	<!--cylinder length="0.154" radius="0.053" /-->
-            		<mesh filename="package://mp500lwa4d_description/meshes/mp500/SICK-S300.STL" />
+                			<!--cylinder length="0.154" radius="0.053" /-->
+            				<mesh filename="package://mp500lwa4d_description/meshes/mp500/SICK-S300.STL" />
 				</geometry>
 				<material name="Gazebo/Yellow" />
   			</visual>
   			<collision>
-				<origin xyz="0 0 0" rpy="3.14 0 -1.57" />
+				<origin xyz="0 0 -0.04" rpy="3.14 0 -1.57" />
 				<geometry>
-	  			<cylinder length="0.154" radius="0.053" />
+					<mesh filename="package://mp500lwa4d_description/meshes/mp500/SICK-S300.STL" />
+	  				<!--cylinder length="0.154" radius="0.053" /-->
 				</geometry>
   			</collision>
